Commit message: add: simple urg settings

File: urdf/minibot_middle_01.xacro (robot description, xacro)
@@ -1,8 +1,8 @@
 <?xml version="1.0"?>
 <robot xmlns:xacro="http://www.ros.org/wiki/xacro" name="minibot_light_01">
-  <xacro:property name="body_d" value="0.24" />
-  <xacro:property name="body_w" value="0.24" />
-  <xacro:property name="body_h" value="0.158" />
-  <xacro:property name="body_offset_x" value="-0.05" />
+  <xacro:property name="body_d" value="0.205" />
+  <xacro:property name="body_w" value="0.285" />
+  <xacro:property name="body_h" value="0.1703" />
+  <xacro:property name="body_offset_x" value="-0.045" />
   <xacro:property name="body_offset_z" value="${body_h/2}" />
   <link name="base_link">
@@ -26,8 +26,8 @@
   <xacro:property name="laser_w" value="0.06" />
   <xacro:property name="laser_h" value="0.06" />
-  <xacro:property name="laser_x" value="0.03" />
-  <xacro:property name="laser_z" value="0.0787" />
+  <xacro:property name="laser_x" value="0.04" />
+  <xacro:property name="laser_z" value="0.01" />
   <joint name="laser_joint" type="fixed">
-    <origin xyz="${laser_x} 0 ${laser_z}" rpy="0 0 ${radians(-90)}"/>
+    <origin xyz="${laser_x} 0 ${laser_z}" rpy="${radians(180)} 0 0"/>
     <parent link="base_link"/>
     <child link="base_laser_link"/>

Commit message: change: Maxon motor configuration

File: urdf/minibot_middle_01.xacro (robot description, xacro)
@@ -1,8 +1,8 @@
 <?xml version="1.0"?>
-<robot xmlns:xacro="http://www.ros.org/wiki/xacro" name="minibot_middle_01">
-  <xacro:property name="body_d" value="0.205" />
-  <xacro:property name="body_w" value="0.285" />
-  <xacro:property name="body_h" value="0.1703" />
-  <xacro:property name="body_offset_x" value="-0.045" />
+<robot xmlns:xacro="http://www.ros.org/wiki/xacro" name="minibot_light_01">
+  <xacro:property name="body_d" value="0.315" />
+  <xacro:property name="body_w" value="0.2423" />
+  <xacro:property name="body_h" value="0.162" />
+  <xacro:property name="body_offset_x" value="${0.07-body_d/2}" />
   <xacro:property name="body_offset_z" value="${body_h/2}" />
   <link name="base_link">
